File: power-board.kicad_pcb (KiCad board)
At the start: 2 copper layers, 127 x 76.2 mm, 152 parts, among them Q3000k1 IRLZ44N, Q4000k1 IRLZ44N

Commit message: Add Ground pads on back
The last step before gerber and drill
Parts:
- added GND: TestPoint_Pad_4.0x4.0mm, TestPoint:TestPoint_Pad_4.0x4.0mm, B.Cu at (144.8, 56.5)
- added GND: TestPoint_Pad_4.0x4.0mm, TestPoint:TestPoint_Pad_4.0x4.0mm, B.Cu at (134.6, 56.5)
