File: LED_Board/capstone-led.kicad_pcb (KiCad board)
At the start: 4 copper layers, 127 x 127 mm, 300 parts

Commit message: Final fixes for JLCPCB
Oval holes changed to circular in LED thermal pad
Routing:
- net VCC: track 101.7 -> 117.8 mm
